Commit message: make turtle_rl independent of turtlebot3_description package, disable rviz2, achieve higher chance of success with robot and lidar in gz

File: turtle_rl/urdf/turtlebot3_burger.gazebo.xacro (robot description, xacro)
@@ -27,5 +27,5 @@
             <scan>
                 <horizontal>
-                    <samples>640</samples>
+                    <samples>360</samples>
                     <resolution>1</resolution>
                     <min_angle>-3.14</min_angle>

File: turtle_rl/urdf/turtlebot3_burger.urdf.xacro (robot description, xacro)
@@ -7,6 +7,4 @@
       <xacro:include filename="$(find turtle_rl)/turtlebot3_burger.gazebo.xacro" />
   </xacro:if>
-  <xacro:arg name="namespace" default=""/>
-  <xacro:property name="namespace" value="$(arg namespace)"/>
   <!-- Init colour -->
   <material name="black">
@@ -40,15 +38,15 @@
     <color rgba="1.0 1.0 1.0 1.0"/>
   </material>
-  <link name="${namespace}base_footprint"/>
-  <joint name="${namespace}base_joint" type="fixed">
-    <parent link="${namespace}base_footprint"/>
-    <child link="${namespace}base_link"/>
+  <link name="base_footprint"/>
+  <joint name="base_joint" type="fixed">
+    <parent link="base_footprint"/>
+    <child link="base_link"/>
     <origin xyz="0.0 0.0 0.010" rpy="0 0 0"/>
   </joint>
-  <link name="${namespace}base_link">
+  <link name="base_link">
     <visual>
       <origin xyz="-0.032 0 0.0" rpy="0 0 0"/>
       <geometry>
-        <mesh filename="package://turtlebot3_description/meshes/bases/burger_base.stl" scale="0.001 0.001 0.001"/>
+        <mesh filename="$(find turtle_rl)/meshes/burger_base.stl" scale="0.001 0.001 0.001"/>
       </geometry>
       <material name="light_black"/>
@@ -66,15 +64,15 @@
     </inertial>
   </link>
-  <joint name="${namespace}wheel_left_joint" type="continuous">
-    <parent link="${namespace}base_link"/>
-    <child link="${namespace}wheel_left_link"/>
+  <joint name="wheel_left_joint" type="continuous">
+    <parent link="base_link"/>
+    <child link="wheel_left_link"/>
     <origin xyz="0.0 0.08 0.023" rpy="-1.57 0 0"/>
     <axis xyz="0 0 1"/>
   </joint>
-  <link name="${namespace}wheel_left_link">
+  <link name="wheel_left_link">
     <visual>
       <origin xyz="0 0 0" rpy="1.57 0 0"/>
       <geometry>
-        <mesh filename="package://turtlebot3_description/meshes/wheels/left_tire.stl" scale="0.001 0.001 0.001"/>
+        <mesh filename="$(find turtle_rl)/meshes/left_tire.stl" scale="0.001 0.001 0.001"/>
       </geometry>
       <material name="dark"/>
@@ -92,15 +90,15 @@
     </inertial>
   </link>
-  <joint name="${namespace}wheel_right_joint" type="continuous">
-    <parent link="${namespace}base_link"/>
-    <child link="${namespace}wheel_right_link"/>
+  <joint name="wheel_right_joint" type="continuous">
+    <parent link="base_link"/>
+    <child link="wheel_right_link"/>
     <origin xyz="0.0 -0.080 0.023" rpy="-1.57 0 0"/>
     <axis xyz="0 0 1"/>
   </joint>
-  <link name="${namespace}wheel_right_link">
+  <link name="wheel_right_link">
     <visual>
       <origin xyz="0 0 0" rpy="1.57 0 0"/>
       <geometry>
-        <mesh filename="package://turtlebot3_description/meshes/wheels/right_tire.stl" scale="0.001 0.001 0.001"/>
+        <mesh filename="$(find turtle_rl)/meshes/right_tire.stl" scale="0.001 0.001 0.001"/>
       </geometry>
       <material name="dark"/>
@@ -118,10 +116,10 @@
     </inertial>
   </link>
-  <joint name="${namespace}caster_back_joint" type="fixed">
-    <parent link="${namespace}base_link"/>
-    <child link="${namespace}caster_back_link"/>
+  <joint name="caster_back_joint" type="fixed">
+    <parent link="base_link"/>
+    <child link="caster_back_link"/>
     <origin xyz="-0.081 0 -0.004" rpy="-1.57 0 0"/>
   </joint>
-  <link name="${namespace}caster_back_link">
+  <link name="caster_back_link">
     <collision>
       <origin xyz="0 0.001 0" rpy="0 0 0"/>
@@ -136,20 +134,20 @@
     </inertial>
   </link>
-  <joint name="${namespace}imu_joint" type="fixed">
-    <parent link="${namespace}base_link"/>
-    <child link="${namespace}imu_link"/>
+  <joint name="imu_joint" type="fixed">
+    <parent link="base_link"/>
+    <child link="imu_link"/>
     <origin xyz="-0.032 0 0.068" rpy="0 0 0"/>
   </joint>
-  <link name="${namespace}imu_link"/>
-  <joint name="${namespace}scan_joint" type="fixed">
-    <parent link="${namespace}base_link"/>
-    <child link="${namespace}base_scan"/>
+  <link name="imu_link"/>
+  <joint name="scan_joint" type="fixed">
+    <parent link="base_link"/>
+    <child link="base_scan"/>
     <origin xyz="-0.032 0 0.172" rpy="0 0 0"/>
   </joint>
-  <link name="${namespace}base_scan">
+  <link name="base_scan">
     <visual>
       <origin xyz="0 0 0.0" rpy="0 0 0"/>
       <geometry>
-        <mesh filename="package://turtlebot3_description/meshes/sensors/lds.stl" scale="0.001 0.001 0.001"/>
+        <mesh filename="$(find turtle_rl)/meshes/lds.stl" scale="0.001 0.001 0.001"/>
       </geometry>
       <material name="dark"/>
