Commit message: change base link collision from box to cylinder

File: turtle_rl/urdf/turtlebot3_burger.urdf.xacro (robot description, xacro)
@@ -7,4 +7,5 @@
       <xacro:include filename="$(find turtle_rl)/turtlebot3_burger.gazebo.xacro" />
   </xacro:if>
+  <xacro:property name="collision_radius" value="0.11"/>
   <!-- Init colour -->
   <material name="black">
@@ -55,5 +56,5 @@
       <origin xyz="-0.032 0 0.070" rpy="0 0 0"/>
       <geometry>
-        <box size="0.140 0.140 0.143"/>
+        <cylinder length="0.143" radius="${collision_radius}"/>
       </geometry>
     </collision>

Commit message: add contact sensor to all fences and obstacles

File: turtle_rl/urdf/turtlebot3_burger.urdf.xacro (robot description, xacro)
@@ -56,5 +56,6 @@
       <origin xyz="-0.032 0 0.070" rpy="0 0 0"/>
       <geometry>
-        <cylinder length="0.143" radius="${collision_radius}"/>
+        <box size="0.140 0.140 0.143"/>
+        <!--<cylinder length="0.143" radius="${collision_radius}"/>-->
       </geometry>
     </collision>

Commit message: change turtlebot collision from box to cylinder, fix a function in map_env

File: turtle_rl/urdf/turtlebot3_burger.urdf.xacro (robot description, xacro)
@@ -56,6 +56,6 @@
       <origin xyz="-0.032 0 0.070" rpy="0 0 0"/>
       <geometry>
-        <box size="0.140 0.140 0.143"/>
-        <!--<cylinder length="0.143" radius="${collision_radius}"/>-->
+        <!--<box size="0.140 0.140 0.143"/>-->
+        <cylinder length="0.11" radius="${collision_radius}"/>
       </geometry>
     </collision>
